File: solo2.sch (KiCad schematic (older format))
At the start: 12 parts, among them P1 USB_C_Plug, SW1 FSUSB42

Commit message: add missing schematics and rename
Parts:
- R10, R2, R3: symbol solo2-rescue:R-Device-solo-A-rescue -> solo2-rescue:R-Device-solo-A-rescue-solo2-rescue
- Z1: symbol solo2-rescue:D_Zener_x2_KCom_AAK-Device-solo-A-rescue -> solo2-rescue:D_Zener_x2_KCom_AAK-Device-solo-A-rescue-solo2-rescue
Changed lines of the file:
@@
 	3650 3650 3800 3650
 $Comp
-L solo2-rescue:R-Device-solo-A-rescue R?
+L solo2-rescue:R-Device-solo-A-rescue-solo2-rescue R?
 U 1 1 5DF57FC3
 P 2500 1550
@@
 $EndComp
 $Comp
-L solo2-rescue:R-Device-solo-A-rescue R?
+L solo2-rescue:R-Device-solo-A-rescue-solo2-rescue R?
 U 1 1 5DF62B4A
 P 3000 1850
@@
 TOP_D+
 $Comp
-L solo2-rescue:D_Zener_x2_KCom_AAK-Device-solo-A-rescue Z1
+L solo2-rescue:D_Zener_x2_KCom_AAK-Device-solo-A-rescue-solo2-rescue Z1
 U 1 1 5E38FEB4
 P 3900 4750
@@
 S 5600 1750 3300 2100
 U 5DDFB633
-F0 "solo" 50
-F1 "solo.sch" 50
+F0 "module" 50
+F1 "module.sch" 50
 F2 "5V" I L 5600 2900 50
 F3 "GND" I L 5600 3050 50
@@
 	2450 4750 2450 4550
 $Comp
-L solo2-rescue:R-Device-solo-A-rescue R?
+L solo2-rescue:R-Device-solo-A-rescue-solo2-rescue R?
 U 1 1 5E65EF73
 P 2850 4700
